File: sch/player.sch (KiCad schematic (older format))
At the start: 1 part

Commit message: schematic add
Parts:
- added AE1: Antenna, Connector_Wire:SolderWirePad_1x01_SMD_1x2mm, symbol Device:Antenna
- added C1, C3, C? (x3): 10uF, Capacitor_SMD:C_0805_2012Metric, symbol Device:C
- added C27: 22pF, Capacitor_SMD:C_0603_1608Metric_Pad1.05x0.95mm_HandSolder, symbol Device:C
- added C28: 1pF, Capacitor_SMD:C_0603_1608Metric_Pad1.05x0.95mm_HandSolder, symbol Device:C
- added C29, C31: 1.5pF, Capacitor_SMD:C_0603_1608Metric_Pad1.05x0.95mm_HandSolder, symbol Device:C
- added C30: 100pF, Capacitor_SMD:C_0603_1608Metric_Pad1.05x0.95mm_HandSolder, symbol Device:C
- added C32: 12pF, Capacitor_SMD:C_0603_1608Metric_Pad1.05x0.95mm_HandSolder, symbol Device:C
- added C33: 3.3pF, Capacitor_SMD:C_0603_1608Metric_Pad1.05x0.95mm_HandSolder, symbol Device:C
- added C34: 47pF, Capacitor_SMD:C_0603_1608Metric_Pad1.05x0.95mm_HandSolder, symbol Device:C
- added C? (x2): 68nF, Capacitor_SMD:C_0805_2012Metric, symbol Device:C
- added C? (x2): 1nF, Capacitor_SMD:C_0805_2012Metric, symbol Device:C
- added C?: 220p, symbol Device:C
- added C? (x5): 1uF, Capacitor_SMD:C_0805_2012Metric, symbol Device:C
- added C? (x2): 100uF, symbol Device:C_Polarized
- added C? (x8): 0.1uF, Capacitor_SMD:C_0603_1608Metric_Pad1.05x0.95mm_HandSolder, symbol Device:C
- added C?: 10uF, Capacitor_SMD:C_0603_1608Metric_Pad1.05x0.95mm_HandSolder, symbol Device:C
- added C? (x2): 0.1uF, Capacitor_SMD:C_0805_2012Metric, symbol Device:C
- added D1: ME2149, Package_SO:SO-8_3.9x4.9mm_P1.27mm, symbol native:ME2149
- added D2, D?: 1N5822, Diode_SMD:D_SMA, symbol Diode:1N5822
- added J4: USB_B, Connector_Wire:SolderWire-0.127sqmm_1x05_P3.7mm_D0.48mm_OD1mm, symbol Connector:USB_B
- added J?: OLED, symbol Connector_Generic:Conn_01x14
- added L1, L2, L5, L6: 12nH, Inductor_SMD:L_0603_1608Metric_Pad1.05x0.95mm_HandSolder, symbol Device:L
- added L1: 4.7mH, Inductor_SMD:L_7.3x7.3_H4.5, symbol Device:L
- added L3, L4: 18nH, Inductor_SMD:L_0603_1608Metric_Pad1.05x0.95mm_HandSolder, symbol Device:L
- added L7: 3.3nH, Inductor_SMD:L_0603_1608Metric_Pad1.05x0.95mm_HandSolder, symbol Device:L
- added R10: 10K, Resistor_SMD:R_0805_2012Metric_Pad1.15x1.40mm_HandSolder, symbol Device:R
- added R18, R19: 22, Resistor_SMD:R_0805_2012Metric_Pad1.15x1.40mm_HandSolder, symbol Device:R
- added R2: 1k, Resistor_SMD:R_0805_2012Metric, symbol Device:R
- added R20: 1K5, Resistor_SMD:R_0805_2012Metric_Pad1.15x1.40mm_HandSolder, symbol Device:R
- added R3: 6k, Resistor_SMD:R_0805_2012Metric, symbol Device:R
- added R? (x4): 680, Resistor_SMD:R_0805_2012Metric, symbol Device:R
- added R? (x2): 1,5k, Resistor_SMD:R_0805_2012Metric, symbol Device:R
- added R?: 1, symbol Device:R
- added R?: 18k, symbol Device:R
- added R?: 11k, symbol Device:R
- added R?: 560k, symbol Device:R
- added U4: CC1101, belkin:cc1101, symbol native:CC1101
- added U? (x3): LM358, symbol Amplifier_Operational:LM358
- added U?: PCM1754DBQR, DBQ16, symbol native:PCM1754DBQR
- added U?: MC33063AD, Package_SO:SOIC-8_3.9x4.9mm_P1.27mm, symbol Regulator_Switching:MC33063AD
- added U?: LM4811, Package_SO:TSSOP-10_3x3mm_P0.5mm, symbol Amplifier_Audio:LM4811
Connections:
- net +3V3: now reaches U?.1 (VBAT)
- net +3V3: now also U?.13 (VDDA), U?.19 (VDD), U?.32 (VDD), U?.48 (VDD), U?.64 (VDD), C?.1, C?.1, C?.1, C?.1, C?.1, C?.1, C?.2, D?.1 (K), J?.5 (Pin_5), J?.8 (Pin_8), R20.2, R?.2, U?.2 (SwE)
- net GND: now reaches U?.12 (VSSA)
- net GND: now also U?.18 (VSS), U?.31 (VSS), U?.47 (VSS), U?.63 (VSS), C1.1, C27.2, C29.1, C3.1, C30.2, C33.2, C?.1, C?.1, C?.1, C?.1, C?.1, C?.2, C?.2, C?.2, C?.2, C?.2, C?.2, C?.2, C?.2, C?.2, C?.2, C?.2, C?.2, D1.2 (GND), D?.2 (A), J4.4 (GND), J4.5 (Shield), J?.7 (Pin_7), R10.1, R3.2, R?.2, U4.16 (GND), U4.19 (GND), U?.13 (DEMP), U?.14 (MUTE), U?.15 (FMT), U?.4 (CLOCK), U?.4 (DGND), U?.4 (V-), U?.5 (GND), U?.6 (UP/DN), U?.7 (SHDN)
- net I2S_WS: now reaches U?.33 (PB12)
- net I2S_WS: now also U?.3 (LRCK)
- net I2S_CK: now reaches U?.34 (PB13)
- net I2S_CK: now also U?.1 (BCK)
- net I2S_SD: now reaches U?.36 (PB15)
- net I2S_SD: now also U?.2 (DATA)
- net I2S_MCK: now reaches U?.37 (PC6)
- net I2S_MCK: now also U?.16 (SCK)
- new net: J4.3 (D+), R18.1, R20.1
- new net: J4.2 (D-), R19.1
- new net: C?.2, C?.2, R?.1, U?.1
- new net: C?.1, R?.2, U?.2 (-)
- new net: C?.2, U?.10 (VCOM), U?.3 (+), U?.5 (+)
- new net: C?.1, R?.2, U?.6 (-)
- new net: C?.2, C?.2, R?.1, U?.7
- new net: R?.1, U?.7 (VOUTL)
- new net: R?.1, U?.8 (VOUTR)
- new net: C?.1, U?.9 (AGND)
- new net: C?.2, R?.1, R?.2, R?.2 (x2)
- new net: L1.2, U4.12 (RF_P)
- new net: L2.2, U4.13 (RF_N)
- new net: R10.2, U4.17 (RBIAS)
- new net: C27.1, U4.5 (DCOUPL)
- new net: C28.1, C29.2, L1.1, L4.2
- new net: C28.2, C31.2, L2.1, L3.2
- new net: C30.1, L3.1
- new net: C31.1, L4.1, L6.2
- new net: C33.1, L5.2, L6.1
- new net: C32.2, C34.2, L5.1
- new net: AE1.1 (A), C32.1, L7.1
- new net: C34.1, L7.2
- new net: C1.2, D1.3 (CE), D1.5 (VDD), D1.6 (VDD), L1.1
- new net: D1.4 (FB), R2.2, R3.1
- new net: D1.7 (LX), D1.8 (LX), D2.2 (A), L1.2
- new net: R?.1, U?.1 (SwC), U?.7 (Ipk), U?.8 (DC)
- new net: C?.1, U?.3 (TC)
- new net: R?.1, U?.4 (GND)
- new net: R?.1, R?.2, U?.5 (Vfb)
- new net: C?.1, U?.1 (VOUT1)
- new net: C?.1, U?.2 (VIN1)
- new net: C?.2, U?.3 (BYPASS)
- new net: C?.1, U?.8 (VIN2)
- new net: C?.1, U?.9 (VOUT2)
- new net: C?.1, J?.1 (Pin_1)
- new net: J?.12 (Pin_12), R?.1
- new net: C?.1, J?.13 (Pin_13)
- new net: C?.1, C?.2, J?.14 (Pin_14)
- new net: C?.2, J?.2 (Pin_2)
- new net: C?.1, J?.3 (Pin_3)
- new net: C?.2, J?.4 (Pin_4)
- new net +5V: C3.2, C?.1, C?.1, C?.1, D2.1 (K), J4.1 (VBUS), R2.1, R?.2, U?.10 (VDD), U?.6 (VCC), U?.6 (Vin), U?.8 (V+)
- new net D_RST: J?.9 (Pin_9)
- new net D_SCL: J?.10 (Pin_10)
- new net D_SDA: J?.11 (Pin_11)
- new net MISO: U4.2 (SO(GDO1))
- new net MOSI: U4.20 (SI)
- new net NSS: U4.7 (CSn)
- new net SCK: U4.1 (SCLK)
- new net USB_DM: R19.2
- new net USB_DP: R18.2
- new net VCC: U4.11 (AVDD), U4.14 (AVDD), U4.15 (AVDD), U4.18 (DGUARD), U4.4 (DVDD), U4.9 (AVDD)
- no-connect marks 0 -> 8
Other:
- moved on the sheet: U?
