File: sch/player.sch (KiCad schematic (older format))
At the start: 123 parts, among them J1 OLED, J2 USB_B, J3 Micro_SD_Card, J5 SWD, Q1 AO3400, Q2 AO3400, Q3 2SC3583, Q4 AO3400, Q5 DTD114E, SW1 RIGHT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

Commit message: sound front end scenario
Parts:
- J4: renamed from J?; footprint (none) -> local:uefang
Changed lines of the file:
@@
 	3000 1100 3000 4700
 $Comp
-L Connector:AudioJack3 J?
+L Connector:AudioJack3 J4
 U 1 1 6346FB50
 P 10900 5450
-F 0 "J?" H 10620 5475 50  0000 R CNN
+F 0 "J4" H 10620 5475 50  0000 R CNN
 F 1 "AudioJack3" H 10620 5384 50  0000 R CNN
-F 2 "" H 10900 5450 50  0001 C CNN
+F 2 "local:uefang" H 10900 5450 50  0001 C CNN
 F 3 "~" H 10900 5450 50  0001 C CNN
 	1    10900 5450
