File: sch/player_4pin.sch (KiCad schematic (older format))
At the start: 123 parts, among them J1 OLED, J2 USB_B, J3 Micro_SD_Card, J5 SWD, Q1 AO3400, Q2 AO3400, Q3 2SC3583, Q4 AO3400, Q5 DTD114E, SW1 RIGHT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

Commit message: soundcard test board
Parts:
- removed J?: AudioJack3, symbol Connector:AudioJack3
- added J4: AudioJack4, Connector_Audio:Jack_3.5mm_PJ320D_Horizontal, symbol Connector:AudioJack4
Connections:
- net GND: now also J4.R2
- net at C40.2, R21.2: now also J4.S
- net at C39.2: now also J4.T
- net at C38.2: now also J4.R1
Changed lines of the file:
@@
 	5600 4150 5600 5200
 Wire Wire Line
+	10700 5250 10650 5250
+Wire Wire Line
+	10650 5250 10650 4350
+Connection ~ 10650 4350
+Wire Wire Line
 	10650 5350 10700 5350
 Wire Wire Line
@@
 Wire Wire Line
 	10550 5550 10700 5550
+$Comp
+L Connector:AudioJack4 J4
+U 1 1 61E9F2A6
+P 10900 5350
+F 0 "J4" H 10750 5550 50  0000 R CNN
+F 1 "AudioJack4" H 11000 5000 50  0000 R CNN
+F 2 "Connector_Audio:Jack_3.5mm_PJ320D_Horizontal" H 10900 5350 50  0001 C CNN
+F 3 "~" H 10900 5350 50  0001 C CNN
+	1    10900 5350
+	-1   0    0    -1
+$EndComp
 Wire Wire Line
 	7250 4600 7250 5700
@@
 Wire Wire Line
 	1150 6350 1150 6500
+Wire Bus Line
+	5200 3500 9850 3500
+Wire Bus Line
+	5200 6200 10300 6200
+Wire Bus Line
+	650  4750 5100 4750
+Wire Bus Line
+	8050 1150 8050 3450
+Wire Bus Line
+	9900 2450 9900 3450
+Wire Bus Line
+	3600 1000 3600 4700
+Wire Bus Line
+	600  2600 600  6600
+Wire Bus Line
+	5150 1750 5150 7600
+Wire Bus Line
+	3000 1100 3000 4700
 Connection ~ 1150 6500
 Wire Wire Line
 	1150 6500 1800 6500
-Wire Bus Line
-	5200 3500 9850 3500
-Wire Bus Line
-	650  4750 5100 4750
-Wire Bus Line
-	5200 6200 10300 6200
-Wire Bus Line
-	8050 1150 8050 3450
-Wire Bus Line
-	9900 2450 9900 3450
-Wire Bus Line
-	3600 1000 3600 4700
-Wire Bus Line
-	600  2600 600  6600
-Wire Bus Line
-	5150 1750 5150 7600
-Wire Bus Line
-	3000 1100 3000 4700
-$Comp
-L Connector:AudioJack3 J?
-U 1 1 6346FB50
-P 10900 5450
-F 0 "J?" H 10620 5475 50  0000 R CNN
-F 1 "AudioJack3" H 10620 5384 50  0000 R CNN
-F 2 "" H 10900 5450 50  0001 C CNN
-F 3 "~" H 10900 5450 50  0001 C CNN
-	1    10900 5450
-	-1   0    0    -1
-$EndComp
 $EndSCHEMATC
