File: sch/player.kicad_pcb (KiCad board)
At the start: 2 copper layers, 100 parts, among them J2 USB_B, Q1 AO3400, Q2 AO3400, Q3 2SC3583, SW1 RIGHT, SW2 volume, SW3 call, SW4 UP, SW5 DN, SW6 LEFT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

Commit message: add micro and audio checked
Parts:
- added BT1: AAA_Cell, Connector_PinHeader_2.54mm:PinHeader_2x01_P2.54mm_Vertical, F.Cu at (85.8, 64.1)
- added C15: 10uF, Capacitor_SMD:C_0805_2012Metric, F.Cu at (122.4, 163.1)
- added C45: 1uF, Capacitor_SMD:C_0805_2012Metric, F.Cu at (168.4, 162.9)
- added J1: OLED, local:display_14p, F.Cu at (197.6, 95.4)
- added J3: Micro_SD_Card, Connector_Card:microSD_HC_Hirose_DM3BT-DSF-PEJS, F.Cu at (72.2, 156.4)
- added J4: AudioJack4, Connector_Audio:Jack_3.5mm_PJ320D_Horizontal, F.Cu at (129.5, 163.7)
- added J5: SWD, local:3WIRE_PADS, F.Cu at (89.4, 118.5)
- added MK1: Mic, Capacitor_THT:CP_Radial_D5.0mm_P2.50mm, F.Cu at (171.3, 164.9)
- added Q4: AO3400, Package_TO_SOT_SMD:SOT-23, F.Cu at (179.1, 151.8)
- added R25: 100k, Resistor_SMD:R_0402_1005Metric, F.Cu at (162.9, 158.7)
- added R26: 33R, Resistor_SMD:R_0402_1005Metric, F.Cu at (98.3, 164.6)
- added R27: 33R, Resistor_SMD:R_0402_1005Metric, F.Cu at (99.4, 164.6)
- added R28: 10k, Resistor_SMD:R_0402_1005Metric, F.Cu at (120.0, 157.6)
- added R29: 10k, Resistor_SMD:R_0402_1005Metric, F.Cu at (119.0, 167.7)
- added R30: 10k, Resistor_SMD:R_0402_1005Metric, F.Cu at (120.4, 159.1)
- added R31: 10k, Resistor_SMD:R_0402_1005Metric, F.Cu at (119.5, 166.2)
- added R32: 10k, Resistor_SMD:R_0402_1005Metric, F.Cu at (157.2, 167.3)
- added R33: 10k, Resistor_SMD:R_0402_1005Metric, F.Cu at (170.2, 152.2)
- added U7: CC1101, local:cc1101, F.Cu at (161.5, 125.0)
- C23: footprint Capacitor_SMD:C_0805_2012Metric -> Capacitor_SMD:C_0402_1005Metric
- C24, C25, C26, C27, C28: footprint Capacitor_SMD:C_0805_2012Metric -> Capacitor_SMD:C_0603_1608Metric
- C29, C30: value 68nF -> 0.33uF; footprint Capacitor_SMD:C_0805_2012Metric -> Capacitor_SMD:C_0603_1608Metric
- C32, C33: value 1nF -> 470p; footprint Capacitor_SMD:C_0805_2012Metric -> Capacitor_SMD:C_0603_1608Metric
- L2: footprint Inductor_SMD:L_7.3x7.3_H4.5 -> Inductor_SMD:L_1206_3216Metric
- R1, R2, R20, R22, R23, R24, R8, R9: footprint Capacitor_SMD:C_0402_1005Metric -> Resistor_SMD:R_0402_1005Metric
- R10, R21, R4: footprint Resistor_SMD:R_0805_2012Metric -> Resistor_SMD:R_0402_1005Metric
- R11, R12, R13, R14: value 680 -> 33R; footprint Resistor_SMD:R_0805_2012Metric -> Resistor_SMD:R_0402_1005Metric
- R15, R16: value 1,5k -> 10k; footprint Resistor_SMD:R_0805_2012Metric -> Resistor_SMD:R_0402_1005Metric
- SW2: footprint Button_Switch_THT:SW_PUSH_6mm -> local:mouse_encoder
- U9: value LM4811 -> LM4810; footprint Package_SO:TSSOP-10_3x3mm_P0.5mm -> Package_SO:TSSOP-8_3x3mm_P0.65mm
- moved C30 141.5 mm to (110.0, 169.4)
- moved C13 133.8 mm to (102.4, 163.4)
- moved R13 127.3 mm to (115.0, 157.1), turned to 180 degrees
- moved C12 125.9 mm to (116.6, 163.8), turned to 90 degrees
- moved C39 123.4 mm to (121.9, 167.9)
- moved C33 123.2 mm to (113.2, 167.4)
- moved C36 122.5 mm to (117.7, 158.6)
- moved C37 122.4 mm to (167.7, 158.2), turned to 90 degrees
- moved R11 121.7 mm to (115.0, 156.1), turned to 180 degrees
- moved R19 121.0 mm to (161.4, 168.7)
- moved C29 119.6 mm to (111.5, 156.4)
- moved U3 118.6 mm to (113.2, 162.9), turned to 270 degrees
- moved R12 114.5 mm to (115.5, 169.6), turned to 180 degrees
- moved U8 107.7 mm to (106.8, 163.8)
- moved C31 107.5 mm to (110.0, 167.7)
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Connections:
- C32 pad 2: /RDA_R -> Net-(C32-Pad2)
- C33 pad 2: /RDA_L -> Net-(C33-Pad2)
- C34 pad 2: /RDA_R -> Net-(C32-Pad2)
- C35 pad 2: /RDA_L -> Net-(C33-Pad2)
- R13 pad 1: /RDA_R -> Net-(C32-Pad2)
- R14 pad 1: /RDA_L -> Net-(C33-Pad2)
- U1 pad 35: Net-(U1-Pad35) -> /MIC_ON
- U3 pad 1: /RDA_R -> Net-(C32-Pad2)
- U3 pad 7: /RDA_L -> Net-(C33-Pad2)
- U8 pad 5: Net-(U8-Pad5) -> GND
- U8 pad 7: Net-(R12-Pad1) -> Net-(R11-Pad1)
- U8 pad 8: Net-(R11-Pad1) -> Net-(R12-Pad1)
- U9 pad 2: Net-(C34-Pad1) -> Net-(R28-Pad2)
- U9 pad 5: GND -> /SND_ON
- U9 pad 6: GND -> Net-(R29-Pad2)
- U9 pad 7: GND -> Net-(C39-Pad1)
- U9 pad 8: Net-(C35-Pad1) -> +5V
Routing:
- net GND: track 0.00 -> 99.7 mm
- net +5V: track 0.00 -> 41.2 mm, vias 0 -> 3
- net +3V3: track 0.00 -> 37.8 mm, vias 0 -> 4
- net Net-(R11-Pad1): track 0.00 -> 27.6 mm, vias 0 -> 2
- net Net-(R12-Pad1): track 0.00 -> 20.2 mm, vias 0 -> 2
- net Net-(C31-Pad2): track 0.00 -> 13.6 mm, vias 0 -> 2
- net /I2S_MCK: track 0.00 -> 10.4 mm
- net Net-(C33-Pad2): track 0.00 -> 5.36 mm
- net Net-(C32-Pad2): track 0.00 -> 4.81 mm
- net Net-(C26-Pad2): track 0.00 -> 4.49 mm
- net Net-(C30-Pad2): track 0.00 -> 4.33 mm
- net Net-(C24-Pad2): track 0.00 -> 4.23 mm
- net /I2S_CK: track 0.00 -> 4.03 mm
- net Net-(C38-Pad1): track 0.00 -> 3.43 mm
- net /RF_MISO: track 0.00 -> 3.42 mm
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
Commit message: soundcard test board
Parts:
- added AE2: Antenna, Connector_Wire:SolderWirePad_1x01_SMD_1x2mm, F.Cu at (126.0, 83.7)
- added Q5: DTD114E, Package_TO_SOT_SMD:SOT-23, F.Cu at (89.5, 33.8)
- added R34: 100k, Resistor_SMD:R_0402_1005Metric, F.Cu at (126.5, 77.0)
- added R35: 100k, Resistor_SMD:R_0402_1005Metric, F.Cu at (85.9, 33.8)
- BT1, C14, C21, C22, C9, D1, D2, D3, D4, L1, L2, Q1, R1, R2, R3, R4, R5, R6, U2, U5, U6: moved to B.Cu
- C2, C3, C5, C6: value 0.1uF -> 22p
- J4: value AudioJack4 -> AudioJack3; footprint Connector_Audio:Jack_3.5mm_PJ320D_Horizontal -> local:uefang; moved to B.Cu
- moved J1 140.2 mm to (70.9, 35.4), turned to 90 degrees
- moved C6 108.1 mm to (54.4, 109.6)
- moved C3 107.7 mm to (54.7, 114.1)
- moved C16 107.0 mm to (68.1, 38.7), turned to 180 degrees
- moved R7 104.0 mm to (68.0, 36.5), turned to 90 degrees
- moved C18 103.5 mm to (68.1, 39.8), turned to 180 degrees
- moved C20 102.3 mm to (67.7, 32.8), turned to 270 degrees
- moved C19 102.3 mm to (69.5, 29.8), turned to 180 degrees
- moved R5 94.6 mm to (80.0, 32.8), turned to 180 degrees
- moved C21 93.2 mm to (81.5, 27.4), turned to 90 degrees
- moved Q1 92.6 mm to (78.5, 30.0), turned to 180 degrees
- moved C22 92.6 mm to (84.6, 30.2)
- moved C17 92.4 mm to (70.8, 41.0)
- moved R1 92.4 mm to (81.4, 29.7)
- moved R19 88.3 mm to (154.4, 80.6), turned to 270 degrees
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Connections:
- C22 pad 2: +3V3 -> Net-(C22-Pad2)
- C42 pad 1: GND -> /ANT
- C43 pad 1: GND -> /ANT_IN
- C43 pad 2: GND -> Net-(C43-Pad2)
- C44 pad 1: GND -> /ANT
- D3 pad 1: +3V3 -> Net-(C22-Pad2)
- J4 pad S: Net-(C40-Pad2) -> GND
- L7 pad 1: GND -> /ANT
- Q1 pad 1: /CRG_PWM -> Net-(Q1-Pad1)
- Q2 pad 1: GND -> Net-(Q2-Pad1)
- Q3 pad 3: GND -> Net-(C43-Pad2)
- R1 pad 1: /CRG_PWM -> Net-(Q1-Pad1)
- R2 pad 1: /Vbat_FB -> Net-(Q1-Pad1)
- R2 pad 2: /BAT_DIS -> /CRG_PWM
- R22 pad 1: GND -> Net-(Q2-Pad1)
- R23 pad 2: GND -> Net-(C43-Pad2)
- R24 pad 1: +5V -> +3V3
- U1 pad 2: /BAT_DIS -> Net-(U1-Pad2)
- U1 pad 62: GND -> Net-(U1-Pad62)
- U2 pad 3: /BAT_DIS -> Net-(Q5-Pad3)
- U5 pad 3: /BAT_DIS -> Net-(Q5-Pad3)
- U6 pad 3: +3V3 -> Net-(C22-Pad2)
Routing:
- net GND: track 99.7 -> 379.8 mm, vias 0 -> 2
- net +3V3: track 37.8 -> 185.0 mm, vias 4 -> 12
- net /Vbat_FB: track 0.00 -> 35.7 mm, vias 0 -> 1
- net /USB_VBUS: track 0.00 -> 32.9 mm, vias 0 -> 1
- net Net-(Q5-Pad3): track 0.00 -> 29.0 mm, vias 0 -> 2
- net Net-(C39-Pad2): track 0.00 -> 28.7 mm, vias 0 -> 1
- net +5V: track 41.2 -> 62.4 mm, vias 3 -> 7
- net Net-(C5-Pad2): track 0.00 -> 17.0 mm
- net /RDA_CLK: track 0.00 -> 15.7 mm
- net Net-(C22-Pad2): track 0.00 -> 12.7 mm
- net /USB_DM: track 0.00 -> 11.6 mm
- net /ADC_MIC: track 0.00 -> 11.3 mm
- net Net-(C2-Pad2): track 0.00 -> 11.3 mm
- net /USB_DP: track 0.00 -> 10.1 mm
- net Net-(D1-Pad2): track 0.00 -> 9.66 mm
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- added copper zone on F.Cu, net GND

Commit message: sound front end scenario
Parts:
- moved C11 53.8 mm to (51.0, 80.4)
- moved C25 53.8 mm to (62.0, 76.9)
- moved C26 53.8 mm to (62.0, 79.9)
- moved L3 53.8 mm to (62.0, 78.4)
- moved L4 53.8 mm to (62.0, 81.5)
- moved U7 53.8 mm to (56.8, 80.4)
- moved AE1 53.8 mm to (67.3, 82.4)
- moved C23 53.8 mm to (52.3, 82.3)
- moved C24 53.8 mm to (62.1, 83.0)
- moved C27 53.8 mm to (64.4, 77.6)
- moved C28 53.8 mm to (65.1, 83.0)
- moved L5 53.8 mm to (65.9, 80.7)
- moved L6 53.8 mm to (64.3, 80.7)
- moved R10 53.8 mm to (57.3, 76.6)
- moved C15 33.2 mm to (155.4, 126.5)
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Routing:
- net GND: track 379.8 -> 406.9 mm
- net +3V3: track 185.0 -> 178.5 mm
- net /RF_MOSI: track 0.00 -> 3.96 mm
- net Net-(C39-Pad2): track 28.7 -> 26.1 mm
